Commit message: change sumshit

File: urdf/quadruped.urdf (robot description, URDF)
Before this commit: robot mjbots_quad, 14 links, 13 joints
Links:
- added link bl_tip_link
- added link br_tip_link
- added link tl_tip_link
- added link tr_tip_link
Joints:
- added joint bl_leg_to_tip: type fixed, parent bl_leg_link, child bl_tip_link, origin xyz=0 -0.99207 -1.1797 rpy=0 0 0
- added joint br_leg_to_tip: type fixed, parent br_leg_link, child br_tip_link, origin xyz=0 -0.99207 -1.1797 rpy=0 0 0
- added joint tl_leg_to_tip: type fixed, parent tl_leg_link, child tl_tip_link, origin xyz=0 -0.99207 -1.1797 rpy=0 0 0
- added joint tr_leg_to_tip: type fixed, parent tr_leg_link, child tr_tip_link, origin xyz=0 -0.99207 -1.1797 rpy=0 0 0

Commit message: forward and kinematic works, trajectory perfect

File: urdf/quadruped.urdf (robot description, URDF)
Before this commit: robot mjbots_quad, 18 links, 17 joints
Joints:
- joint bl_leg_joint: limit lower=-1.57 upper=1.57 effort=1000 velocity=10 -> lower=-3.14 upper=3.14 effort=100 velocity=10; origin xyz=0.1446 0.7442 -1.2971 rpy=0 0 0 -> xyz=0.1446 0 -1.2971 rpy=0 0 0
- joint bl_shoulder_joint: limit lower=-1.57 upper=1.57 effort=1000 velocity=10 -> lower=-3.14 upper=3.14 effort=100 velocity=10; origin xyz=-0.66731 -1.2 -0.03 rpy=0 0 0 -> xyz=-0.63527 -1.2 -0.03 rpy=0 0 0
- joint bl_thigh_joint: limit lower=-1.57 upper=1.57 effort=1000 velocity=10 -> lower=-3.14 upper=3.14 effort=100 velocity=10
- joint br_leg_joint: limit lower=-1.57 upper=1.57 effort=1000 velocity=10 -> lower=-3.14 upper=3.14 effort=100 velocity=10; origin xyz=-0.1303 0.7467 -1.2935 rpy=0 0 0 -> xyz=-0.1446 0 -1.2971 rpy=0 0 0
- joint br_shoulder_joint: limit lower=-1.57 upper=1.57 effort=1000 velocity=10 -> lower=-3.14 upper=3.14 effort=100 velocity=10
- joint br_thigh_joint: limit lower=-1.57 upper=1.57 effort=1000 velocity=10 -> lower=-3.14 upper=3.14 effort=100 velocity=10; origin xyz=1.12423 -0.6152 0.001 rpy=0 0 0 -> xyz=1.120 -0.6203 0.022 rpy=0 0 0
- joint tl_leg_joint: limit lower=-1.57 upper=1.57 effort=1000 velocity=10 -> lower=-3.14 upper=3.14 effort=100 velocity=10; origin xyz=0.1283 0.7444 -1.2941 rpy=0 0 0 -> xyz=0.1256 0 -1.295 rpy=0 0 0
- joint tl_shoulder_joint: limit lower=-1.57 upper=1.57 effort=1000 velocity=10 -> lower=-3.14 upper=3.14 effort=100 velocity=10
- joint tl_thigh_joint: limit lower=-1.57 upper=1.57 effort=1000 velocity=10 -> lower=-3.14 upper=3.14 effort=100 velocity=10
- joint tr_leg_joint: limit lower=-1.57 upper=1.57 effort=1000 velocity=10 -> lower=-3.14 upper=3.14 effort=100 velocity=10; origin xyz=-0.1256 0.7477 -1.295 rpy=0 0 0 -> xyz=-0.1256 0 -1.295 rpy=0 0 0
- joint tr_shoulder_joint: limit lower=-1.57 upper=1.57 effort=1000 velocity=10 -> lower=-3.14 upper=3.14 effort=100 velocity=10; origin xyz=0.63315 1.1646 -0.0414 rpy=0 0 0 -> xyz=0.6667 1.1462 -0.0414 rpy=0 0 0
- joint tr_thigh_joint: limit lower=-1.57 upper=1.57 effort=1000 velocity=10 -> lower=-3.14 upper=3.14 effort=100 velocity=10; origin xyz=1.13265 0.6225 -0.0006 rpy=0 0 0 -> xyz=1.1059 0.639 -0.0012 rpy=0 0 0
