Commit message: added fosmc and ai critic

File: urdf/quadruped.urdf (robot description, URDF)
Before this commit: robot mjbots_quad, 18 links, 17 joints
Links:
- link base_link: geometry collision mesh filename=package://quins_ros2/meshes/QUAD_BODY_C.stl scale=0.1 0.1 0.1; visual mesh filename=package://quins_ros2/meshes/QUAD_BODY.stl scale=0.1 0.1 0.1
- link bl_leg_link: geometry collision mesh filename=package://quins_ros2/meshes/QUAD_BL_LEG_C.stl scale=0.1 0.1 0.1; visual mesh filename=package://quins_ros2/meshes/QUAD_BL_LEG.stl scale=0.1 0.1 0.1
- link bl_shoulder_link: geometry collision mesh filename=package://quins_ros2/meshes/QUAD_BL_SHOULDER_C.stl scale=0.1 0.1 0.1; visual mesh filename=package://quins_ros2/meshes/QUAD_BL_SHOULDER.stl scale=0.1 0.1 0.1
- link bl_thigh_link: geometry collision mesh filename=package://quins_ros2/meshes/QUAD_BL_THIGH_C.stl scale=0.1 0.1 0.1; visual mesh filename=package://quins_ros2/meshes/QUAD_BL_THIGH.stl scale=0.1 0.1 0.1
- link br_leg_link: geometry collision mesh filename=package://quins_ros2/meshes/QUAD_BR_LEG_C.stl scale=0.1 0.1 0.1; visual mesh filename=package://quins_ros2/meshes/QUAD_BR_LEG.stl scale=0.1 0.1 0.1
- link br_shoulder_link: geometry collision mesh filename=package://quins_ros2/meshes/QUAD_BR_SHOULDER_C.stl scale=0.1 0.1 0.1; visual mesh filename=package://quins_ros2/meshes/QUAD_BR_SHOULDER.stl scale=0.1 0.1 0.1
- link br_thigh_link: geometry collision mesh filename=package://quins_ros2/meshes/QUAD_BR_THIGH_C.stl scale=0.1 0.1 0.1; visual mesh filename=package://quins_ros2/meshes/QUAD_BR_THIGH.stl scale=0.1 0.1 0.1
- link tl_leg_link: geometry collision mesh filename=package://quins_ros2/meshes/QUAD_TL_LEG_C.stl scale=0.1 0.1 0.1; visual mesh filename=package://quins_ros2/meshes/QUAD_TL_LEG.stl scale=0.1 0.1 0.1
- link tl_shoulder_link: geometry collision mesh filename=package://quins_ros2/meshes/QUAD_TL_SHOULDER_C.stl scale=0.1 0.1 0.1; visual mesh filename=package://quins_ros2/meshes/QUAD_TL_SHOULDER.stl scale=0.1 0.1 0.1
- link tl_thigh_link: geometry collision mesh filename=package://quins_ros2/meshes/QUAD_TL_THIGH_C.stl scale=0.1 0.1 0.1; visual mesh filename=package://quins_ros2/meshes/QUAD_TL_THIGH.stl scale=0.1 0.1 0.1
- link tr_leg_link: geometry collision mesh filename=package://quins_ros2/meshes/QUAD_TR_LEG_C.stl scale=0.1 0.1 0.1; visual mesh filename=package://quins_ros2/meshes/QUAD_TR_LEG.stl scale=0.1 0.1 0.1
- link tr_shoulder_link: geometry collision mesh filename=package://quins_ros2/meshes/QUAD_TR_SHOULDER_C.stl scale=0.1 0.1 0.1; visual mesh filename=package://quins_ros2/meshes/QUAD_TR_SHOULDER.stl scale=0.1 0.1 0.1
- link tr_thigh_link: geometry collision mesh filename=package://quins_ros2/meshes/QUAD_TR_THIGH_C.stl scale=0.1 0.1 0.1; visual mesh filename=package://quins_ros2/meshes/QUAD_TR_THIGH.stl scale=0.1 0.1 0.1

Commit message: actually good wbc mpc with new model

File: urdf/quadruped.urdf (robot description, URDF)
Before this commit: robot mjbots_quad, 17 links, 16 joints
Links:
- removed link bl_leg_link
- removed link bl_shoulder_link
- removed link bl_thigh_link
- removed link bl_tip_link
- removed link br_leg_link
- removed link br_shoulder_link
- removed link br_thigh_link
- removed link br_tip_link
- removed link tl_leg_link
- removed link tl_shoulder_link
- removed link tl_thigh_link
- removed link tl_tip_link
- removed link tr_leg_link
- removed link tr_shoulder_link
- removed link tr_thigh_link
- removed link tr_tip_link
- added link LF_FOOT; collision sphere radius=0.014
- added link LF_HIP, mass 0.7; visual mesh filename=package://quins_ros2/meshes/QUINS_LF_HIP.stl scale=0.001 0.001 0.001
- added link LF_SHANK, mass 0.3; visual mesh filename=package://quins_ros2/meshes/QUINS_LF_SHANK.stl scale=0.001 0.001 0.001
- added link LF_THIGH, mass 0.8; visual mesh filename=package://quins_ros2/meshes/QUINS_LF_THIGH.stl scale=0.001 0.001 0.001
- added link LH_FOOT; collision sphere radius=0.014
- added link LH_HIP, mass 0.7; visual mesh filename=package://quins_ros2/meshes/QUINS_LH_HIP.stl scale=0.001 0.001 0.001
- added link LH_SHANK, mass 0.3; visual mesh filename=package://quins_ros2/meshes/QUINS_LH_SHANK.stl scale=0.001 0.001 0.001
- added link LH_THIGH, mass 0.8; visual mesh filename=package://quins_ros2/meshes/QUINS_LH_THIGH.stl scale=0.001 0.001 0.001
- added link RF_FOOT; collision sphere radius=0.014
- added link RF_HIP, mass 0.7; visual mesh filename=package://quins_ros2/meshes/QUINS_RF_HIP.stl scale=0.001 0.001 0.001
- added link RF_SHANK, mass 0.3; visual mesh filename=package://quins_ros2/meshes/QUINS_RF_SHANK.stl scale=0.001 0.001 0.001
- added link RF_THIGH, mass 0.8; visual mesh filename=package://quins_ros2/meshes/QUINS_RF_THIGH.stl scale=0.001 0.001 0.001
- added link RH_FOOT; collision sphere radius=0.014
- added link RH_HIP, mass 0.7; visual mesh filename=package://quins_ros2/meshes/QUINS_RH_HIP.stl scale=0.001 0.001 0.001
- added link RH_SHANK, mass 0.3; visual mesh filename=package://quins_ros2/meshes/QUINS_RH_SHANK.stl scale=0.001 0.001 0.001
- added link RH_THIGH, mass 0.8; visual mesh filename=package://quins_ros2/meshes/QUINS_RH_THIGH.stl scale=0.001 0.001 0.001
- link base_link: mass 5.0 -> 3.0; geometry collision mesh filename=package://quins_ros2/meshes/QUINS_BODY.stl scale=0.001 0.001 0.001; visual mesh filename=package://quins_ros2/meshes/QUINS_BODY.stl scale=0.001 0.001 0.001
Joints:
- removed joint bl_leg_joint
- removed joint bl_leg_to_tip
- removed joint bl_shoulder_joint
- removed joint bl_thigh_joint
- removed joint br_leg_joint
- removed joint br_leg_to_tip
- removed joint br_shoulder_joint
- removed joint br_thigh_joint
- removed joint tl_leg_joint
- removed joint tl_leg_to_tip
- removed joint tl_shoulder_joint
- removed joint tl_thigh_joint
- removed joint tr_leg_joint
- removed joint tr_leg_to_tip
- removed joint tr_shoulder_joint
- removed joint tr_thigh_joint
- added joint LF_HAA: type revolute, parent base_link, child LF_HIP, origin xyz=-0.157 0.060 0 rpy=0 0 0, axis 1 0 0, limit lower=-3.14 upper=3.14 effort=100 velocity=10
- added joint LF_HFE: type revolute, parent LF_HIP, child LF_THIGH, origin xyz=-0.053 0.030 0 rpy=0 0 0, axis 0 -1 0, limit lower=-3.14 upper=3.14 effort=100 velocity=10
- added joint LF_KFE: type revolute, parent LF_THIGH, child LF_SHANK, origin xyz=0 0.172 -0.17985 rpy=0 0 0, axis 0 -1 0, limit lower=-3.14 upper=3.14 effort=100 velocity=10
- added joint LF_SHANK_TO_FOOT: type fixed, parent LF_SHANK, child LF_FOOT, origin xyz=0.040 0.0245 -0.23015 rpy=0 0 0
- added joint LH_HAA: type revolute, parent base_link, child LH_HIP, origin xyz=0.157 0.060 0 rpy=0 0 0, axis 1 0 0, limit lower=-3.14 upper=3.14 effort=100 velocity=10
- added joint LH_HFE: type revolute, parent LH_HIP, child LH_THIGH, origin xyz=0.053 0.030 0 rpy=0 0 0, axis 0 -1 0, limit lower=-3.14 upper=3.14 effort=100 velocity=10
- added joint LH_KFE: type revolute, parent LH_THIGH, child LH_SHANK, origin xyz=0 0.172 -0.17985 rpy=0 0 0, axis 0 -1 0, limit lower=-3.14 upper=3.14 effort=100 velocity=10
- added joint LH_SHANK_TO_FOOT: type fixed, parent LH_SHANK, child LH_FOOT, origin xyz=0.040 0.0245 -0.23015 rpy=0 0 0
- added joint RF_HAA: type revolute, parent base_link, child RF_HIP, origin xyz=-0.157 -0.060 0 rpy=0 0 0, axis 1 0 0, limit lower=-3.14 upper=3.14 effort=100 velocity=10
- added joint RF_HFE: type revolute, parent RF_HIP, child RF_THIGH, origin xyz=-0.053 -0.030 0 rpy=0 0 0, axis 0 -1 0, limit lower=-3.14 upper=3.14 effort=100 velocity=10
- added joint RF_KFE: type revolute, parent RF_THIGH, child RF_SHANK, origin xyz=0 -0.172 -0.17985 rpy=0 0 0, axis 0 -1 0, limit lower=-3.14 upper=3.14 effort=100 velocity=10
- added joint RF_SHANK_TO_FOOT: type fixed, parent RF_SHANK, child RF_FOOT, origin xyz=0.040 -0.0245 -0.23015 rpy=0 0 0
- added joint RH_HAA: type revolute, parent base_link, child RH_HIP, origin xyz=0.157 -0.060 0 rpy=0 0 0, axis 1 0 0, limit lower=-3.14 upper=3.14 effort=100 velocity=10
- added joint RH_HFE: type revolute, parent RH_HIP, child RH_THIGH, origin xyz=0.053 -0.030 0 rpy=0 0 0, axis 0 -1 0, limit lower=-3.14 upper=3.14 effort=100 velocity=10
- added joint RH_KFE: type revolute, parent RH_THIGH, child RH_SHANK, origin xyz=0 -0.172 -0.17985 rpy=0 0 0, axis 0 -1 0, limit lower=-3.14 upper=3.14 effort=100 velocity=10
- added joint RH_SHANK_TO_FOOT: type fixed, parent RH_SHANK, child RH_FOOT, origin xyz=0.040 -0.0245 -0.23015 rpy=0 0 0

Commit message: achieved stable walk between 2 control system
WBC + FOSMC Stable at forward (+x) for over 20s
exposed all FOSMC and WBC required variable for RL Tuning

File: urdf/quadruped.urdf (robot description, URDF)
Before this commit: robot quins, 17 links, 16 joints
Links:
- link LF_FOOT: mass None -> 0.0115
- link LF_HIP: geometry visual mesh filename=package://quins_ros2/meshes/QUINS_LH_HIP.stl scale=0.001 0.001 0.001
- link LF_SHANK: geometry visual mesh filename=package://quins_ros2/meshes/QUINS_LH_SHANK.stl scale=0.001 0.001 0.001
- link LF_THIGH: geometry visual mesh filename=package://quins_ros2/meshes/QUINS_LH_THIGH.stl scale=0.001 0.001 0.001
- link LH_FOOT: mass None -> 0.0115
- link LH_HIP: geometry visual mesh filename=package://quins_ros2/meshes/QUINS_LF_HIP.stl scale=0.001 0.001 0.001
- link LH_SHANK: geometry visual mesh filename=package://quins_ros2/meshes/QUINS_LF_SHANK.stl scale=0.001 0.001 0.001
- link LH_THIGH: geometry visual mesh filename=package://quins_ros2/meshes/QUINS_LF_THIGH.stl scale=0.001 0.001 0.001
- link RF_FOOT: mass None -> 0.0115
- link RF_HIP: geometry visual mesh filename=package://quins_ros2/meshes/QUINS_RH_HIP.stl scale=0.001 0.001 0.001
- link RF_SHANK: geometry visual mesh filename=package://quins_ros2/meshes/QUINS_RH_SHANK.stl scale=0.001 0.001 0.001
- link RF_THIGH: geometry visual mesh filename=package://quins_ros2/meshes/QUINS_RH_THIGH.stl scale=0.001 0.001 0.001
- link RH_FOOT: mass None -> 0.0115
- link RH_HIP: geometry visual mesh filename=package://quins_ros2/meshes/QUINS_RF_HIP.stl scale=0.001 0.001 0.001
- link RH_SHANK: geometry visual mesh filename=package://quins_ros2/meshes/QUINS_RF_SHANK.stl scale=0.001 0.001 0.001
- link RH_THIGH: geometry visual mesh filename=package://quins_ros2/meshes/QUINS_RF_THIGH.stl scale=0.001 0.001 0.001
Joints:
- joint LF_HAA: origin xyz=-0.157 0.060 0 rpy=0 0 0 -> xyz=0.157 0.060 0 rpy=0 0 0
- joint LF_HFE: origin xyz=-0.053 0.030 0 rpy=0 0 0 -> xyz=0.053 0.030 0 rpy=0 0 0
- joint LH_HAA: origin xyz=0.157 0.060 0 rpy=0 0 0 -> xyz=-0.157 0.060 0 rpy=0 0 0
- joint LH_HFE: origin xyz=0.053 0.030 0 rpy=0 0 0 -> xyz=-0.053 0.030 0 rpy=0 0 0
- joint RF_HAA: origin xyz=-0.157 -0.060 0 rpy=0 0 0 -> xyz=0.157 -0.060 0 rpy=0 0 0
- joint RF_HFE: origin xyz=-0.053 -0.030 0 rpy=0 0 0 -> xyz=0.053 -0.030 0 rpy=0 0 0
- joint RH_HAA: origin xyz=0.157 -0.060 0 rpy=0 0 0 -> xyz=-0.157 -0.060 0 rpy=0 0 0
- joint RH_HFE: origin xyz=0.053 -0.030 0 rpy=0 0 0 -> xyz=-0.053 -0.030 0 rpy=0 0 0
